File: CM5_HighSpeed.kicad_sch (KiCad schematic)
At the start: 19 parts, among them J10 690-019-298-412, J12 USB3_A, J16 Conn_01x22_Female, J22 690-019-298-412, J5 Conn_01x22_Female, J6 THD-02-R, U12 RT9742SNGV, U6 AP22653W6

Commit message: Need to fix ERC
Parts:
- removed C12, C13: 100n, Capacitor_SMD:C_0402_1005Metric, symbol Device:C
- removed J10, J22: 690-019-298-412, CM5IO:EDAC 690-019-298-412, symbol CM5IO:HDMI_A_1.4
- removed J6: THD-02-R, Connector_PinHeader_2.54mm:PinHeader_2x02_P2.54mm_Vertical, symbol Connector_Generic:Conn_02x02_Odd_Even
- removed U12: RT9742SNGV, Package_TO_SOT_SMD:TSOT-23_HandSoldering, symbol CM5IO:RT9742SNGV
- added JP1, JP2: SolderJumper_2_Open, symbol Jumper:SolderJumper_2_Open
- renumbered C2 to C3, C3 to C4, C7 to C5, C8 to C6, J5 to J2, J16 to J3, J12 to J4, R12 to R2, R8 to R3, R6 to R4, R7 to R5, U6 to U1
Connections:
- net ID_SC: now also JP1.1 (A)
- net ID_SD: now also JP2.1 (A)
- net SCL1: now also JP1.2 (B)
- net SDA1: now also JP2.2 (B)
- net HDMI0_CEC: no longer names the net of Module1.151 (HDMI0_CEC)
- net HDMI0_CK_N: no longer names the net of Module1.190 (HDMI0_CLK_N)
- net HDMI0_CK_P: no longer names the net of Module1.188 (HDMI0_CLK_P)
- net HDMI0_D0_N: no longer names the net of Module1.184 (HDMI0_TX0_N)
- net HDMI0_D0_P: no longer names the net of Module1.182 (HDMI0_TX0_P)
- net HDMI0_D1_N: no longer names the net of Module1.178 (HDMI0_TX1_N)
- net HDMI0_D1_P: no longer names the net of Module1.176 (HDMI0_TX1_P)
- net HDMI0_D2_N: no longer names the net of Module1.172 (HDMI0_TX2_N)
- net HDMI0_D2_P: no longer names the net of Module1.170 (HDMI0_TX2_P)
- net HDMI0_HOTPLUG: no longer names the net of Module1.153 (HDMI0_HOTPLUG)
- net HDMI0_SCL: no longer names the net of Module1.200 (HDMI0_SCL)
- net HDMI0_SDA: no longer names the net of Module1.199 (HDMI0_SDA)
- net HDMI1_CEC: no longer names the net of Module1.149 (HDMI1_CEC)
- net HDMI1_CK_N: no longer names the net of Module1.166 (HDMI1_CLK_N)
- net HDMI1_CK_P: no longer names the net of Module1.164 (HDMI1_CLK_P)
- net HDMI1_D0_N: no longer names the net of Module1.160 (HDMI1_TX0_N)
- net HDMI1_D0_P: no longer names the net of Module1.158 (HDMI1_TX0_P)
- net HDMI1_D1_N: no longer names the net of Module1.154 (HDMI1_TX1_N)
- net HDMI1_D1_P: no longer names the net of Module1.152 (HDMI1_TX1_P)
- net HDMI1_D2_N: no longer names the net of Module1.148 (HDMI1_TX2_N)
- net HDMI1_D2_P: no longer names the net of Module1.146 (HDMI1_TX2_P)
- net HDMI1_HOTPLUG: no longer names the net of Module1.143 (HDMI1_HOTPLUG)
- net HDMI1_SCL: no longer names the net of Module1.147 (HDMI1_SCL)
- net HDMI1_SDA: no longer names the net of Module1.145 (HDMI1_SDA)
- net PCIE_CLK_N: no longer names the net of Module1.112 (PCIe_CLK_N)
- net PCIE_CLK_P: no longer names the net of Module1.110 (PCIe_CLK_P)
- net PCIE_PWR_EN: no longer names the net of Module1.106 (PCIE_PWR_EN)
- net PCIE_RX_N: no longer names the net of Module1.118 (PCIe_RX_N)
- net PCIE_RX_P: no longer names the net of Module1.116 (PCIe_RX_P)
- net PCIE_TX_N: no longer names the net of Module1.124 (PCIe_TX_N)
- net PCIE_TX_P: no longer names the net of Module1.122 (PCIe_TX_P)
- net PCIE_nCLKREQ: no longer names the net of Module1.102 (PCIe_nCLKREQ)
- net PCIE_nRST: no longer names the net of Module1.109 (PCIe_nRST)
- net PCIE_nWAKE: no longer names the net of Module1.104 (PCIE_nWAKE)
- no-connect marks 4 -> 35

Commit message: schematic review
Other:
- company: Copyright © 2024 Raspberry Pi Ltd. -> Astrosystems
- title: Compute Module 5 IO Board - CM5 - Highspeed -> CM4/5 - Highspeed
Changed lines of the file:
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@@
 	(paper "A4")
 	(title_block
-		(title "Compute Module 5 IO Board - CM5 - Highspeed")
+		(title "CM4/5 - Highspeed")
+		(date "2025-08-26")
 		(rev "1")
-		(company "Copyright © 2024 Raspberry Pi Ltd.")
-		(comment 1 "www.raspberrypi.com")
+		(company "Astrosystems")
+		(comment 1 "Designed By - C.P")
 	)
 	(text "CM4 Camera"

Commit message: updated files
Connections:
- no-connect marks 35 -> 36
Changed lines of the file:
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@@
+	)
+	(no_connect
+		(at 99.06 35.56)
 	)
 	(no_connect
