File: USB-UART-converter.kicad_sch (KiCad schematic)
At the start: 29 parts, among them J8 430450600, J9 USB_B, Q4 FDV301N, Q5 FDV301N, Q6 FDV301N, U7 74HC02, U8 CP2102N-Axx-xQFN28

Commit message: schematic review
Other:
- company: (none) -> Astrosystems
- title: (none) -> VAL364 Circuit
Changed lines of the file:
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@@
 	(generator_version "9.0")
 	(paper "A4")
+	(title_block
+		(title "VAL364 Circuit")
+		(date "2025-08-26")
+		(rev "1")
+		(company "Astrosystems")
+		(comment 1 "Designed By - C.P")
+	)
 	(text "RX"
 		(exclude_from_sim no)
